File: IGN6.kicad_sch (KiCad schematic)
At the start: 24 parts

Commit message: zmiana 1
Parts:
- renumbered F6 to F5, F5 to F6
Changed lines of the file:
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@@
 		(shape input)
 		(at 190.5 97.79 0)
+		(fields_autoplaced yes)
 		(effects
 			(font
@@
 		(shape output)
 		(at 113.03 64.77 180)
+		(fields_autoplaced yes)
 		(effects
 			(font
@@
 		(shape output)
 		(at 113.03 120.65 180)
+		(fields_autoplaced yes)
 		(effects
 			(font
@@
 		(shape input)
 		(at 143.51 97.79 0)
+		(fields_autoplaced yes)
 		(effects
 			(font
@@
 		(shape input)
 		(at 190.5 125.73 0)
+		(fields_autoplaced yes)
 		(effects
 			(font
@@
 		(shape output)
 		(at 160.02 120.65 180)
+		(fields_autoplaced yes)
 		(effects
 			(font
@@
 		(shape output)
 		(at 160.02 92.71 180)
+		(fields_autoplaced yes)
 		(effects
 			(font
@@
 		(shape output)
 		(at 113.03 92.71 180)
+		(fields_autoplaced yes)
 		(effects
 			(font
@@
 		(shape input)
 		(at 143.51 125.73 0)
+		(fields_autoplaced yes)
 		(effects
 			(font
@@
 		(shape input)
 		(at 143.51 69.85 0)
+		(fields_autoplaced yes)
 		(effects
 			(font
@@
 		(shape output)
 		(at 160.02 64.77 180)
+		(fields_autoplaced yes)
 		(effects
 			(font
@@
 		(shape input)
 		(at 190.5 69.85 0)
+		(fields_autoplaced yes)
 		(effects
 			(font
@@
 			(project "uaefi"
 				(path "/ac264c30-3e9a-4be2-b97a-9949b68bd497/92c4206f-a69e-4d4d-9308-206d3518e11e"
-					(reference "Q9")
+					(reference "Q3")
 					(unit 1)
 				)
@@
 			(project "uaefi"
 				(path "/ac264c30-3e9a-4be2-b97a-9949b68bd497/92c4206f-a69e-4d4d-9308-206d3518e11e"
-					(reference "R27")
+					(reference "R33")
 					(unit 1)
 				)
@@
 			(project "uaefi"
 				(path "/ac264c30-3e9a-4be2-b97a-9949b68bd497/92c4206f-a69e-4d4d-9308-206d3518e11e"
-					(reference "R17")
+					(reference "R23")
 					(unit 1)
 				)
@@
 			(project "uaefi"
 				(path "/ac264c30-3e9a-4be2-b97a-9949b68bd497/92c4206f-a69e-4d4d-9308-206d3518e11e"
-					(reference "R26")
+					(reference "R32")
 					(unit 1)
 				)
@@
 			(project "uaefi"
 				(path "/ac264c30-3e9a-4be2-b97a-9949b68bd497/92c4206f-a69e-4d4d-9308-206d3518e11e"
-					(reference "R25")
+					(reference "R31")
 					(unit 1)
 				)
@@
 			(project "uaefi"
 				(path "/ac264c30-3e9a-4be2-b97a-9949b68bd497/92c4206f-a69e-4d4d-9308-206d3518e11e"
-					(reference "R18")
+					(reference "R24")
 					(unit 1)
 				)
@@
 			(project "uaefi"
 				(path "/ac264c30-3e9a-4be2-b97a-9949b68bd497/92c4206f-a69e-4d4d-9308-206d3518e11e"
-					(reference "#PWR0101")
+					(reference "#PWR0121")
 					(unit 1)
 				)
@@
 			(project "uaefi"
 				(path "/ac264c30-3e9a-4be2-b97a-9949b68bd497/92c4206f-a69e-4d4d-9308-206d3518e11e"
-					(reference "R20")
+					(reference "R26")
 					(unit 1)
 				)
@@
 			(project "uaefi"
 				(path "/ac264c30-3e9a-4be2-b97a-9949b68bd497/92c4206f-a69e-4d4d-9308-206d3518e11e"
-					(reference "Q7")
+					(reference "Q1")
 					(unit 1)
 				)
@@
 			(project "uaefi"
 				(path "/ac264c30-3e9a-4be2-b97a-9949b68bd497/92c4206f-a69e-4d4d-9308-206d3518e11e"
-					(reference "#PWR0104")
+					(reference "#PWR0124")
 					(unit 1)
 				)
@@
 			(project "uaefi"
 				(path "/ac264c30-3e9a-4be2-b97a-9949b68bd497/92c4206f-a69e-4d4d-9308-206d3518e11e"
-					(reference "R19")
+					(reference "R25")
 					(unit 1)
 				)
@@
 			(project "uaefi"
 				(path "/ac264c30-3e9a-4be2-b97a-9949b68bd497/92c4206f-a69e-4d4d-9308-206d3518e11e"
-					(reference "Q8")
+					(reference "Q2")
 					(unit 1)
 				)
@@
 			(project "uaefi"
 				(path "/ac264c30-3e9a-4be2-b97a-9949b68bd497/92c4206f-a69e-4d4d-9308-206d3518e11e"
-					(reference "#PWR099")
+					(reference "#PWR0119")
 					(unit 1)
 				)
@@
 		(on_board yes)
 		(dnp no)
-		(property "Reference" "F6"
+		(property "Reference" "F5"
 			(at 139.7 67.31 90)
 			(effects
@@
 			(project "uaefi"
 				(path "/ac264c30-3e9a-4be2-b97a-9949b68bd497/92c4206f-a69e-4d4d-9308-206d3518e11e"
-					(reference "F6")
+					(reference "F5")
 					(unit 1)
 				)
@@
 			(project "uaefi"
 				(path "/ac264c30-3e9a-4be2-b97a-9949b68bd497/92c4206f-a69e-4d4d-9308-206d3518e11e"
-					(reference "Q10")
+					(reference "Q4")
 					(unit 1)
 				)
@@
 			(project "uaefi"
 				(path "/ac264c30-3e9a-4be2-b97a-9949b68bd497/92c4206f-a69e-4d4d-9308-206d3518e11e"
-					(reference "R24")
+					(reference "R30")
 					(unit 1)
 				)
@@
 		(on_board yes)
 		(dnp no)
-		(property "Reference" "F5"
+		(property "Reference" "F6"
 			(at 139.7 95.25 90)
 			(effects
@@
 			(project "uaefi"
 				(path "/ac264c30-3e9a-4be2-b97a-9949b68bd497/92c4206f-a69e-4d4d-9308-206d3518e11e"
-					(reference "F5")
+					(reference "F6")
 					(unit 1)
 				)
@@
 			(project "uaefi"
 				(path "/ac264c30-3e9a-4be2-b97a-9949b68bd497/92c4206f-a69e-4d4d-9308-206d3518e11e"
-					(reference "Q12")
+					(reference "Q6")
 					(unit 1)
 				)
@@
 			(project "uaefi"
 				(path "/ac264c30-3e9a-4be2-b97a-9949b68bd497/92c4206f-a69e-4d4d-9308-206d3518e11e"
-					(reference "R28")
+					(reference "R34")
 					(unit 1)
 				)
@@
 			(project "uaefi"
 				(path "/ac264c30-3e9a-4be2-b97a-9949b68bd497/92c4206f-a69e-4d4d-9308-206d3518e11e"
-					(reference "#PWR0102")
+					(reference "#PWR0122")
 					(unit 1)
 				)
@@
 			(project "uaefi"
 				(path "/ac264c30-3e9a-4be2-b97a-9949b68bd497/92c4206f-a69e-4d4d-9308-206d3518e11e"
-					(reference "R21")
+					(reference "R27")
 					(unit 1)
 				)
@@
 			(project "uaefi"
 				(path "/ac264c30-3e9a-4be2-b97a-9949b68bd497/92c4206f-a69e-4d4d-9308-206d3518e11e"
-					(reference "R23")
+					(reference "R29")
 					(unit 1)
 				)
@@
 			(project "uaefi"
 				(path "/ac264c30-3e9a-4be2-b97a-9949b68bd497/92c4206f-a69e-4d4d-9308-206d3518e11e"
-					(reference "#PWR0103")
+					(reference "#PWR0123")
 					(unit 1)
 				)
@@
 			(project "uaefi"
 				(path "/ac264c30-3e9a-4be2-b97a-9949b68bd497/92c4206f-a69e-4d4d-9308-206d3518e11e"
-					(reference "#PWR0100")
+					(reference "#PWR0120")
 					(unit 1)
 				)
@@
 			(project "uaefi"
 				(path "/ac264c30-3e9a-4be2-b97a-9949b68bd497/92c4206f-a69e-4d4d-9308-206d3518e11e"
-					(reference "R22")
+					(reference "R28")
 					(unit 1)
 				)
@@
 			(project "uaefi"
 				(path "/ac264c30-3e9a-4be2-b97a-9949b68bd497/92c4206f-a69e-4d4d-9308-206d3518e11e"
-					(reference "Q11")
-					(unit 1)
-				)
+					(reference "Q5")
+					(unit 1)
+				)
