File: MAP.kicad_sch (KiCad schematic)
At the start: 2 parts, among them U3 MPX4/MPXH6400_MAP

Commit message: zmiana 1
Parts:
- renumbered U3 to U7
Changed lines of the file:
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@@
 		(shape output)
 		(at 167.64 83.82 0)
+		(fields_autoplaced yes)
 		(effects
 			(font
@@
 			(project "uaefi"
 				(path "/ac264c30-3e9a-4be2-b97a-9949b68bd497/7f618b1f-fe11-49db-a473-d0b521b1fa4f"
-					(reference "#PWR096")
+					(reference "#PWR0116")
 					(unit 1)
 				)
@@
 			(project "uaefi"
 				(path "/ac264c30-3e9a-4be2-b97a-9949b68bd497/7f618b1f-fe11-49db-a473-d0b521b1fa4f"
-					(reference "#PWR098")
+					(reference "#PWR0118")
 					(unit 1)
 				)
@@
 			(project "uaefi"
 				(path "/ac264c30-3e9a-4be2-b97a-9949b68bd497/7f618b1f-fe11-49db-a473-d0b521b1fa4f"
-					(reference "#PWR097")
+					(reference "#PWR0117")
 					(unit 1)
 				)
@@
 			(project "uaefi"
 				(path "/ac264c30-3e9a-4be2-b97a-9949b68bd497/7f618b1f-fe11-49db-a473-d0b521b1fa4f"
-					(reference "C27")
+					(reference "C28")
 					(unit 1)
 				)
@@
 		(dnp no)
 		(fields_autoplaced yes)
-		(property "Reference" "U3"
+		(property "Reference" "U7"
 			(at 142.24 77.47 0)
 			(effects
@@
 			(project "uaefi"
 				(path "/ac264c30-3e9a-4be2-b97a-9949b68bd497/7f618b1f-fe11-49db-a473-d0b521b1fa4f"
-					(reference "U3")
-					(unit 1)
-				)
+					(reference "U7")
+					(unit 1)
+				)
