File: egt.kicad_sch (KiCad schematic)
At the start: 9 parts, among them U4 MAX31855KASA

Commit message: zmiana 1
Parts:
- renumbered D8 to D6, U4 to U8
Changed lines of the file:
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@@
 		(shape input)
 		(at 201.93 68.58 0)
+		(fields_autoplaced yes)
 		(effects
 			(font
@@
 		(shape output)
 		(at 194.31 90.17 0)
+		(fields_autoplaced yes)
 		(effects
 			(font
@@
 		(shape input)
 		(at 194.31 87.63 0)
+		(fields_autoplaced yes)
 		(effects
 			(font
@@
 		(shape input)
 		(at 194.31 95.25 0)
+		(fields_autoplaced yes)
 		(effects
 			(font
@@
 		(shape input)
 		(at 101.6 87.63 180)
+		(fields_autoplaced yes)
 		(effects
 			(font
@@
 		(shape input)
 		(at 101.6 95.25 180)
+		(fields_autoplaced yes)
 		(effects
 			(font
@@
 			(project "uaefi"
 				(path "/ac264c30-3e9a-4be2-b97a-9949b68bd497/ced20183-e5c8-42b4-80bd-35fc70d9313a"
-					(reference "C28")
+					(reference "C29")
 					(unit 1)
 				)
@@
 		(on_board yes)
 		(dnp no)
-		(property "Reference" "U4"
+		(property "Reference" "U8"
 			(at 168.5641 80.01 0)
 			(effects
@@
 			(project "uaefi"
 				(path "/ac264c30-3e9a-4be2-b97a-9949b68bd497/ced20183-e5c8-42b4-80bd-35fc70d9313a"
-					(reference "U4")
+					(reference "U8")
 					(unit 1)
 				)
@@
 			(project "uaefi"
 				(path "/ac264c30-3e9a-4be2-b97a-9949b68bd497/ced20183-e5c8-42b4-80bd-35fc70d9313a"
-					(reference "C32")
+					(reference "C33")
 					(unit 1)
 				)
@@
 			(project "uaefi"
 				(path "/ac264c30-3e9a-4be2-b97a-9949b68bd497/ced20183-e5c8-42b4-80bd-35fc70d9313a"
-					(reference "C30")
+					(reference "C31")
 					(unit 1)
 				)
@@
 		(on_board yes)
 		(dnp no)
-		(property "Reference" "D8"
+		(property "Reference" "D6"
 			(at 120.65 105.41 0)
 			(effects
@@
 			(project "uaefi"
 				(path "/ac264c30-3e9a-4be2-b97a-9949b68bd497/ced20183-e5c8-42b4-80bd-35fc70d9313a"
-					(reference "D8")
+					(reference "D6")
 					(unit 1)
 				)
@@
 			(project "uaefi"
 				(path "/ac264c30-3e9a-4be2-b97a-9949b68bd497/ced20183-e5c8-42b4-80bd-35fc70d9313a"
-					(reference "C31")
+					(reference "C32")
 					(unit 1)
 				)
@@
 		(on_board yes)
 		(dnp no)
-		(property "Reference" "#PWR0109"
+		(property "Reference" "#PWR0129"
 			(at 176.53 83.82 0)
 			(effects
@@
 			(project "uaefi"
 				(path "/ac264c30-3e9a-4be2-b97a-9949b68bd497/ced20183-e5c8-42b4-80bd-35fc70d9313a"
-					(reference "#PWR0109")
+					(reference "#PWR0129")
 					(unit 1)
 				)
@@
 		(on_board yes)
 		(dnp no)
-		(property "Reference" "#PWR0110"
+		(property "Reference" "#PWR0130"
 			(at 189.23 83.82 0)
 			(effects
@@
 			(project "uaefi"
 				(path "/ac264c30-3e9a-4be2-b97a-9949b68bd497/ced20183-e5c8-42b4-80bd-35fc70d9313a"
-					(reference "#PWR0110")
+					(reference "#PWR0130")
 					(unit 1)
 				)
@@
 		(on_board yes)
 		(dnp no)
-		(property "Reference" "#PWR0106"
+		(property "Reference" "#PWR0126"
 			(at 135.89 114.3 0)
 			(effects
@@
 			(project "uaefi"
 				(path "/ac264c30-3e9a-4be2-b97a-9949b68bd497/ced20183-e5c8-42b4-80bd-35fc70d9313a"
-					(reference "#PWR0106")
+					(reference "#PWR0126")
 					(unit 1)
 				)
@@
 		(on_board yes)
 		(dnp no)
-		(property "Reference" "#PWR0107"
+		(property "Reference" "#PWR0127"
 			(at 151.13 114.3 0)
 			(effects
@@
 			(project "uaefi"
 				(path "/ac264c30-3e9a-4be2-b97a-9949b68bd497/ced20183-e5c8-42b4-80bd-35fc70d9313a"
-					(reference "#PWR0107")
+					(reference "#PWR0127")
 					(unit 1)
 				)
@@
 		(on_board yes)
 		(dnp no)
-		(property "Reference" "#PWR0108"
+		(property "Reference" "#PWR0128"
 			(at 166.37 111.76 0)
 			(effects
@@
 			(project "uaefi"
 				(path "/ac264c30-3e9a-4be2-b97a-9949b68bd497/ced20183-e5c8-42b4-80bd-35fc70d9313a"
-					(reference "#PWR0108")
+					(reference "#PWR0128")
 					(unit 1)
 				)
@@
 		(on_board yes)
 		(dnp no)
-		(property "Reference" "#PWR0105"
+		(property "Reference" "#PWR0125"
 			(at 119.38 114.3 0)
 			(effects
@@
 			(project "uaefi"
 				(path "/ac264c30-3e9a-4be2-b97a-9949b68bd497/ced20183-e5c8-42b4-80bd-35fc70d9313a"
-					(reference "#PWR0105")
+					(reference "#PWR0125")
 					(unit 1)
 				)
@@
 			(project "uaefi"
 				(path "/ac264c30-3e9a-4be2-b97a-9949b68bd497/ced20183-e5c8-42b4-80bd-35fc70d9313a"
-					(reference "C29")
-					(unit 1)
-				)
+					(reference "C30")
+					(unit 1)
+				)
