File: gdi4.kicad_sch (KiCad schematic)
At the start: 311 parts, among them J1 Conn_02x02_Odd_Even, J2 FTSH-107-01-F-DV-K, J3 TC2030, J4 Conn_01x06, J5 Conn_01x06, P1 368255-2, P18 Pad, P19 Pad, P2 Pad, P20 Pad, P3 Pad, P36 Pad, P4 Pad, P5 Pad, Q1 BUK9230-100B, Q10 BUK9230-100B, Q11 BUK9230-100B, Q12 BUK9230-100B, Q13 AOD4185, Q14 VND14NV04TR-E, Q15 VND14NV04TR-E, Q16 BUK9230-100B, Q2 BUK9230-100B, Q3 BUK9230-100B, Q4 BUK9230-100B, Q5 BUK9230-100B, Q6 BUK9230-100B, Q7 BUK9230-100B, Q8 BUK9230-100B, Q9 BUK9230-100B, U1 MC33PT2001AE, U2 TJA1051T-3, U3 LM78M05_TO252, U4 74HC14PW,118, U5 XC6206P332MR, U6 MCP6004, U7 STM32F103CBT6, U8 74HC14PW,118, Y1 8MHz, Y2 1MHz

Commit message: zmiana1b
Parts:
- R1, R109, R110, R111, R112, R117, R118, R119, R120, R121, R122, R28, R30, R32, R37, R41, R44, R5, R55, R57, R58, R59, R61, R62, R63, R64, R65, R66, R67, R68, R69, R70, R71, R72, R73, R74, R75, R76, R77, R78, R79, R80, R81, R82, R83, R84, R85, R86, R87, R88, R89, R91: now not fitted
Changed lines of the file:
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@@
 		(in_bom yes)
 		(on_board yes)
-		(dnp no)
+		(dnp yes)
 		(property "Reference" "R67"
 			(at 142.875 122.555 0)
@@
 		(in_bom yes)
 		(on_board yes)
-		(dnp no)
+		(dnp yes)
 		(property "Reference" "R120"
 			(at 216.535 262.89 90)
@@
 		(in_bom yes)
 		(on_board yes)
-		(dnp no)
+		(dnp yes)
 		(property "Reference" "R37"
 			(at 442.595 372.745 0)
@@
 		(in_bom yes)
 		(on_board yes)
-		(dnp no)
+		(dnp yes)
 		(property "Reference" "R110"
 			(at 142.875 150.495 0)
@@
 		(in_bom yes)
 		(on_board yes)
-		(dnp no)
+		(dnp yes)
 		(property "Reference" "R117"
 			(at 208.915 262.89 90)
@@
 		(in_bom yes)
 		(on_board yes)
-		(dnp no)
+		(dnp yes)
 		(property "Reference" "R86"
 			(at 156.21 107.315 0)
@@
 		(in_bom yes)
 		(on_board yes)
-		(dnp no)
+		(dnp yes)
 		(property "Reference" "R66"
 			(at 142.875 244.475 0)
@@
 		(in_bom yes)
 		(on_board yes)
-		(dnp no)
+		(dnp yes)
 		(property "Reference" "R28"
 			(at 217.17 358.14 90)
@@
 		(in_bom yes)
 		(on_board yes)
-		(dnp no)
+		(dnp yes)
 		(property "Reference" "R73"
 			(at 156.21 97.155 0)
@@
 		(in_bom yes)
 		(on_board yes)
-		(dnp no)
+		(dnp yes)
 		(property "Reference" "R61"
 			(at 142.875 221.615 0)
@@
 		(in_bom yes)
 		(on_board yes)
-		(dnp no)
+		(dnp yes)
 		(property "Reference" "R81"
 			(at 534.035 233.045 0)
@@
 		(in_bom yes)
 		(on_board yes)
-		(dnp no)
+		(dnp yes)
 		(property "Reference" "R68"
 			(at 146.05 160.655 0)
@@
 		(in_bom yes)
 		(on_board yes)
-		(dnp no)
+		(dnp yes)
 		(property "Reference" "R118"
 			(at 211.455 262.89 90)
@@
 		(in_bom yes)
 		(on_board yes)
-		(dnp no)
+		(dnp yes)
 		(property "Reference" "R1"
 			(at 142.875 239.395 0)
@@
 		(in_bom yes)
 		(on_board yes)
-		(dnp no)
+		(dnp yes)
 		(property "Reference" "R32"
 			(at 224.79 358.14 90)
@@
 		(in_bom yes)
 		(on_board yes)
-		(dnp no)
+		(dnp yes)
 		(property "Reference" "R87"
 			(at 156.21 328.295 0)
@@
 		(in_bom yes)
 		(on_board yes)
-		(dnp no)
+		(dnp yes)
 		(property "Reference" "R59"
 			(at 142.875 127.635 0)
@@
 		(in_bom yes)
 		(on_board yes)
-		(dnp no)
+		(dnp yes)
 		(property "Reference" "R121"
 			(at 517.525 132.715 0)
@@
 		(in_bom yes)
 		(on_board yes)
-		(dnp no)
+		(dnp yes)
 		(property "Reference" "R57"
 			(at 142.875 120.015 0)
@@
 		(in_bom yes)
 		(on_board yes)
-		(dnp no)
+		(dnp yes)
 		(property "Reference" "R76"
 			(at 157.48 351.155 0)
@@
 		(in_bom yes)
 		(on_board yes)
-		(dnp no)
+		(dnp yes)
 		(property "Reference" "R109"
 			(at 142.875 147.955 0)
@@
 		(in_bom yes)
 		(on_board yes)
-		(dnp no)
+		(dnp yes)
 		(property "Reference" "R119"
 			(at 213.995 262.89 90)
@@
 		(in_bom yes)
 		(on_board yes)
-		(dnp no)
+		(dnp yes)
 		(property "Reference" "R44"
 			(at 450.215 165.735 0)
@@
 		(in_bom yes)
 		(on_board yes)
-		(dnp no)
+		(dnp yes)
 		(property "Reference" "R58"
 			(at 142.875 125.095 0)
@@
 		(in_bom yes)
 		(on_board yes)
-		(dnp no)
+		(dnp yes)
 		(property "Reference" "R70"
 			(at 156.21 89.535 0)
@@
 		(in_bom yes)
 		(on_board yes)
-		(dnp no)
+		(dnp yes)
 		(property "Reference" "R80"
 			(at 534.035 200.025 0)
@@
 		(in_bom yes)
 		(on_board yes)
-		(dnp no)
+		(dnp yes)
 		(property "Reference" "R79"
 			(at 157.48 366.395 0)
@@
 		(in_bom yes)
 		(on_board yes)
-		(dnp no)
+		(dnp yes)
 		(property "Reference" "R62"
 			(at 142.875 231.775 0)
@@
 		(in_bom yes)
 		(on_board yes)
-		(dnp no)
+		(dnp yes)
 		(property "Reference" "R63"
 			(at 142.875 226.695 0)
@@
 		(in_bom yes)
 		(on_board yes)
-		(dnp no)
+		(dnp yes)
 		(property "Reference" "R74"
 			(at 156.21 99.695 0)
@@
 		(in_bom yes)
 		(on_board yes)
-		(dnp no)
+		(dnp yes)
 		(property "Reference" "R88"
 			(at 235.585 210.82 0)
@@
 		(in_bom yes)
 		(on_board yes)
-		(dnp no)
+		(dnp yes)
 		(property "Reference" "R71"
 			(at 156.21 92.075 0)
@@
 		(in_bom yes)
 		(on_board yes)
-		(dnp no)
+		(dnp yes)
 		(property "Reference" "R41"
 			(at 442.595 403.225 0)
@@
 		(in_bom yes)
 		(on_board yes)
-		(dnp no)
+		(dnp yes)
 		(property "Reference" "R91"
 			(at 235.585 215.9 0)
@@
 		(in_bom yes)
 		(on_board yes)
-		(dnp no)
+		(dnp yes)
 		(property "Reference" "R85"
 			(at 156.21 104.775 0)
@@
 		(in_bom yes)
 		(on_board yes)
-		(dnp no)
+		(dnp yes)
 		(property "Reference" "R55"
 			(at 450.215 168.275 0)
@@
 		(in_bom yes)
 		(on_board yes)
-		(dnp no)
+		(dnp yes)
 		(property "Reference" "R78"
 			(at 157.48 361.315 0)
@@
 		(in_bom yes)
 		(on_board yes)
-		(dnp no)
+		(dnp yes)
 		(property "Reference" "R5"
 			(at 213.36 358.14 90)
@@
 		(in_bom yes)
 		(on_board yes)
-		(dnp no)
+		(dnp yes)
 		(property "Reference" "R69"
 			(at 146.05 165.735 0)
@@
 		(in_bom yes)
 		(on_board yes)
-		(dnp no)
+		(dnp yes)
 		(property "Reference" "R30"
 			(at 220.98 358.14 90)
@@
 		(in_bom yes)
 		(on_board yes)
-		(dnp no)
+		(dnp yes)
 		(property "Reference" "R82"
 			(at 534.035 235.585 0)
@@
 		(in_bom yes)
 		(on_board yes)
-		(dnp no)
+		(dnp yes)
 		(property "Reference" "R112"
 			(at 142.875 201.295 0)
@@
 		(in_bom yes)
 		(on_board yes)
-		(dnp no)
+		(dnp yes)
 		(property "Reference" "R122"
 			(at 517.525 135.255 0)
@@
 		(in_bom yes)
 		(on_board yes)
-		(dnp no)
+		(dnp yes)
 		(property "Reference" "R84"
 			(at 156.21 102.235 0)
@@
 		(in_bom yes)
 		(on_board yes)
-		(dnp no)
+		(dnp yes)
 		(property "Reference" "R89"
 			(at 235.585 213.36 0)
@@
 		(in_bom yes)
 		(on_board yes)
-		(dnp no)
+		(dnp yes)
 		(property "Reference" "R65"
 			(at 142.875 241.935 0)
@@
 		(in_bom yes)
 		(on_board yes)
-		(dnp no)
+		(dnp yes)
 		(property "Reference" "R75"
 			(at 156.21 333.375 0)
@@
 		(in_bom yes)
 		(on_board yes)
-		(dnp no)
+		(dnp yes)
 		(property "Reference" "R72"
 			(at 156.21 94.615 0)
@@
 		(in_bom yes)
 		(on_board yes)
-		(dnp no)
+		(dnp yes)
 		(property "Reference" "R83"
 			(at 534.035 250.825 0)
@@
 		(in_bom yes)
 		(on_board yes)
-		(dnp no)
+		(dnp yes)
 		(property "Reference" "R77"
 			(at 157.48 356.235 0)
@@
 		(in_bom yes)
 		(on_board yes)
-		(dnp no)
+		(dnp yes)
 		(property "Reference" "R111"
 			(at 142.875 198.755 0)
@@
 		(in_bom yes)
 		(on_board yes)
-		(dnp no)
+		(dnp yes)
 		(property "Reference" "R64"
 			(at 142.875 234.315 0)

Commit message: zmiana3
Parts:
- R1, R117, R118, R119, R120, R122, R28, R30, R32, R41, R44, R5, R55, R80, R81, R82, R83, R88: now fitted
- R109, R110, R111, R112, R121, R37, R57, R58, R59, R61, R62, R63, R64, R65, R66, R67, R68, R69, R70, R71, R72, R73, R74, R75, R76, R77, R78, R79, R84, R85, R86, R87, R89, R91: value Jumper-Pad-Pad -> DNP; now fitted

Commit message: zmiana 10k
Parts:
- R100, R105, R106, R107, R108, R2, R34, R35, R56, R60, R92, R93, R95, R96, R97, R98, R99: value 10k -> 10K
Changed lines of the file:
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@@
 			)
 		)
-		(property "Value" "10k"
+		(property "Value" "10K"
 			(at 240.03 273.05 0)
 			(effects
@@
 			)
 		)
-		(property "Value" "10k"
+		(property "Value" "10K"
 			(at 240.03 275.59 0)
 			(effects
@@
 			)
 		)
-		(property "Value" "10k"
+		(property "Value" "10K"
 			(at 261.62 176.53 0)
 			(effects
@@
 			)
 		)
-		(property "Value" "10k"
+		(property "Value" "10K"
 			(at 318.1966 119.6371 90)
 			(effects
@@
 			)
 		)
-		(property "Value" "10k"
+		(property "Value" "10K"
 			(at 233.68 372.11 0)
 			(effects
@@
 			)
 		)
-		(property "Value" "10k"
+		(property "Value" "10K"
 			(at 261.62 171.45 0)
 			(effects
@@
 			)
 		)
-		(property "Value" "10k"
+		(property "Value" "10K"
 			(at 176.5916 120.2721 90)
 			(effects
@@
 			)
 		)
-		(property "Value" "10k"
+		(property "Value" "10K"
 			(at 261.62 168.91 0)
 			(effects
@@
 			)
 		)
-		(property "Value" "10k"
+		(property "Value" "10K"
 			(at 240.03 280.67 0)
 			(effects
@@
 			)
 		)
-		(property "Value" "10k"
+		(property "Value" "10K"
 			(at 233.68 377.19 0)
 			(effects
@@
 			)
 		)
-		(property "Value" "10k"
+		(property "Value" "10K"
 			(at 233.68 374.65 0)
 			(effects
@@
 			)
 		)
-		(property "Value" "10k"
+		(property "Value" "10K"
 			(at 261.62 173.99 0)
 			(effects
@@
 			)
 		)
-		(property "Value" "10k"
+		(property "Value" "10K"
 			(at 261.62 214.63 0)
 			(effects
@@
 			)
 		)
-		(property "Value" "10k"
+		(property "Value" "10K"
 			(at 240.03 278.13 0)
 			(effects
@@
 			)
 		)
-		(property "Value" "10k"
+		(property "Value" "10K"
 			(at 318.1966 95.5071 90)
 			(effects
@@
 			)
 		)
-		(property "Value" "10k"
+		(property "Value" "10K"
 			(at 261.62 217.17 0)
 			(effects
@@
 			)
 		)
-		(property "Value" "10k"
+		(property "Value" "10K"
 			(at 233.68 379.73 0)
 			(effects
