File: uaefi.kicad_sch (KiCad schematic)
At the start: 72 parts, among them J1 Conn_02x02_Odd_Even, J1 USB_B_Mini, J1 USB_C, J10 5569-16A2, J11 Conn_02x02_Odd_Even, J12 Conn_02x02_Odd_Even, J13 Conn_02x02_Odd_Even, J14 Conn_02x02_Odd_Even, J15 Conn_02x02_Odd_Even, J16 Conn_02x02_Odd_Even, J17 Conn_01x06, J17 Conn_02x02_Odd_Even, J18 Conn_02x02_Odd_Even, J19 Conn_02x02_Odd_Even, J2 5569-20A2, J20 Conn_02x02_Odd_Even, J21 Conn_02x02_Odd_Even, J22 Conn_02x02_Odd_Even, J24 Conn_02x02_Odd_Even, J3 5569-06A2, J4 5569-08A2, J5 5569-18A2, J5 Conn_01x05_Male, M1 Module-power_12and5V-0.3, M3 Module-knock-0.2, M3 Module-vr-discrete-0.5, M4 Module-vr-max9924-0.1, M5 Module-wbo-0.5, M6 Module:mega-mcu100/0.3, M7 Module-can-0.1, P1 Pad, P2 Pad, P3 Pad, P4 Pad, P5 Pad, P6 Pad, P7 Pad, P8 Pad, U4 JDY-33

Commit message: zmiana 1
Parts:
- renumbered D2 to D1, D3 to D2, D4 to D3, D5 to D4, G3 to G1, G4 to G2, G1 to G3, G2 to G4, J22 to J1, J12 to J10, J15 to J11, J19 to J12, J11 to J13, J16 to J14, J24 to J15, J20 to J16, J1 to J18, J21 to J19, J13 to J2, J17 to J20, J14 to J3, J10 to J4, J2 to J5, J3 to J6, J4 to J7, J18 to J8, J5 to J9, P5 to P1, P6 to P2, P4 to P3, P3 to P4, P7 to P5, P8 to P6, P1 to P7, P2 to P8
Other:
- added sheet gdi4 (gdi4.kicad_sch)

Commit message: zmiana1b
Parts:
- R38, R39, R4, R41: now not fitted
Changed lines of the file:
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@@
 		(in_bom yes)
 		(on_board yes)
-		(dnp no)
+		(dnp yes)
 		(property "Reference" "R4"
 			(at 132.08 316.23 0)
@@
 		(in_bom yes)
 		(on_board yes)
-		(dnp no)
+		(dnp yes)
 		(property "Reference" "R41"
 			(at 171.45 297.18 0)
@@
 		(in_bom yes)
 		(on_board yes)
-		(dnp no)
+		(dnp yes)
 		(property "Reference" "R39"
 			(at 171.45 292.1 0)
@@
 		(in_bom yes)
 		(on_board yes)
-		(dnp no)
+		(dnp yes)
 		(property "Reference" "R38"
 			(at 171.45 287.02 0)

Commit message: zmiana3
Parts:
- R38, R39, R41: now fitted
- R4: value Jumper-Pad-Pad -> DNP; now fitted
Changed lines of the file:
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@@
 		(in_bom yes)
 		(on_board yes)
-		(dnp yes)
+		(dnp no)
 		(property "Reference" "R4"
 			(at 132.08 316.23 0)
@@
 			)
 		)
-		(property "Value" "Jumper-Pad-Pad"
+		(property "Value" "DNP"
 			(at 127 319.278 0)
 			(effects
@@
 		(in_bom yes)
 		(on_board yes)
-		(dnp yes)
+		(dnp no)
 		(property "Reference" "R41"
 			(at 171.45 297.18 0)
@@
 		(in_bom yes)
 		(on_board yes)
-		(dnp yes)
+		(dnp no)
 		(property "Reference" "R39"
 			(at 171.45 292.1 0)
@@
 		(in_bom yes)
 		(on_board yes)
-		(dnp yes)
+		(dnp no)
 		(property "Reference" "R38"
 			(at 171.45 287.02 0)

Commit message: Zmiana 6.8k
Parts:
- R30: value 6.8k -> 6.8K
Changed lines of the file:
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@@
 			)
 		)
-		(property "Value" "6.8k"
+		(property "Value" "6.8K"
 			(at 64.77 149.86 0)
 			(effects

Commit message: zmiana 10k
Parts:
- R38: value 10k -> 10K
Changed lines of the file:
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@@
 			)
 		)
-		(property "Value" "10k"
+		(property "Value" "10K"
 			(at 200.66 298.45 0)
 			(effects
@@
 			)
 		)
-		(property "Value" "10k"
+		(property "Value" "10K"
 			(at 200.66 288.29 0)
 			(effects
@@
 			)
 		)
-		(property "Value" "10k"
+		(property "Value" "10K"
 			(at 200.66 293.37 0)
 			(effects
